Commit message: [URDF] Update the URDF according to the latest Panda Package

File: data/urdf/panda_default.urdf (robot description, URDF)
Before this commit: robot panda_default, 11 links, 10 joints
Links:
- link panda_link0: geometry collision cylinder length=0.03 radius=0.09; collision sphere radius=0.09
- link panda_link1: geometry collision cylinder length=0.2830 radius=0.09; collision sphere radius=0.09
- link panda_link2: geometry collision cylinder length=0.12 radius=0.09; collision sphere radius=0.09
- link panda_link3: geometry collision cylinder length=0.15 radius=0.09; collision sphere radius=0.09
- link panda_link4: geometry collision cylinder length=0.12 radius=0.09; collision sphere radius=0.09
- link panda_link5: geometry collision cylinder length=0.1 radius=0.09; collision cylinder length=0.14 radius=0.055
- link panda_link6: geometry collision cylinder length=0.08 radius=0.08; collision sphere radius=0.08
- link panda_link7: geometry collision cylinder length=0.14 radius=0.07; collision sphere radius=0.07

File: data/urdf/panda_foot.urdf (robot description, URDF)
Before this commit: robot panda_foot, 12 links, 11 joints
Links:
- link panda_link0: geometry collision cylinder length=0.03 radius=0.09; collision sphere radius=0.09
- link panda_link1: geometry collision cylinder length=0.2830 radius=0.09; collision sphere radius=0.09
- link panda_link2: geometry collision cylinder length=0.12 radius=0.09; collision sphere radius=0.09
- link panda_link3: geometry collision cylinder length=0.15 radius=0.09; collision sphere radius=0.09
- link panda_link4: geometry collision cylinder length=0.12 radius=0.09; collision sphere radius=0.09
- link panda_link5: geometry collision cylinder length=0.1 radius=0.09; collision cylinder length=0.14 radius=0.055
- link panda_link6: geometry collision cylinder length=0.08 radius=0.08; collision sphere radius=0.08
- link panda_link7: geometry collision cylinder length=0.14 radius=0.07; collision sphere radius=0.07

File: data/urdf/panda_hand.urdf (robot description, URDF)
Before this commit: robot panda_hand, 14 links, 13 joints
Links:
- link panda_hand: geometry collision cylinder length=0.1 radius=0.02; collision cylinder length=0.1 radius=0.04
- link panda_leftfinger: geometry visual mesh filename=file://@URDF_DESTINATION@/meshes/visual/finger.dae
- link panda_link0: geometry collision cylinder length=0.03 radius=0.09; collision sphere radius=0.09
- link panda_link1: geometry collision cylinder length=0.2830 radius=0.09; collision sphere radius=0.09
- link panda_link2: geometry collision cylinder length=0.12 radius=0.09; collision sphere radius=0.09
- link panda_link3: geometry collision cylinder length=0.15 radius=0.09; collision sphere radius=0.09
- link panda_link4: geometry collision cylinder length=0.12 radius=0.09; collision sphere radius=0.09
- link panda_link5: geometry collision cylinder length=0.1 radius=0.09; collision cylinder length=0.14 radius=0.055
- link panda_link6: geometry collision cylinder length=0.08 radius=0.08; collision sphere radius=0.08
- link panda_link7: geometry collision cylinder length=0.14 radius=0.07; collision sphere radius=0.07
- link panda_rightfinger: geometry visual mesh filename=file://@URDF_DESTINATION@/meshes/visual/finger.dae

File: data/urdf/panda_pump.urdf (robot description, URDF)
Before this commit: robot panda_pump, 12 links, 11 joints
Links:
- link panda_link0: geometry collision cylinder length=0.03 radius=0.09; collision sphere radius=0.09
- link panda_link1: geometry collision cylinder length=0.2830 radius=0.09; collision sphere radius=0.09
- link panda_link2: geometry collision cylinder length=0.12 radius=0.09; collision sphere radius=0.09
- link panda_link3: geometry collision cylinder length=0.15 radius=0.09; collision sphere radius=0.09
- link panda_link4: geometry collision cylinder length=0.12 radius=0.09; collision sphere radius=0.09
- link panda_link5: geometry collision cylinder length=0.1 radius=0.09; collision cylinder length=0.14 radius=0.055
- link panda_link6: geometry collision cylinder length=0.08 radius=0.08; collision sphere radius=0.08
- link panda_link7: geometry collision cylinder length=0.14 radius=0.07; collision sphere radius=0.07

File: data/xacro/panda.xacro (robot description, xacro)
@@ -29,5 +29,5 @@
         <origin xyz="0 0 0" rpy="0 0 0"/>
         <geometry>
-          <mesh filename="package://${package_name}/meshes/robot_arms/fr3/visual/link0.dae"/>
+          <mesh filename="package://${package_name}/meshes/visual/link0.dae"/>
         </geometry>
         <material name="">
@@ -65,5 +65,5 @@
         <origin xyz="0 0 0" rpy="0 0 0"/>
         <geometry>
-          <mesh filename="package://${package_name}/meshes/robot_arms/fr3/visual/link1.dae"/>
+          <mesh filename="package://${package_name}/meshes/visual/link1.dae"/>
         </geometry>
         <material name="">
@@ -109,5 +109,5 @@
         <origin xyz="0 0 0" rpy="0 0 0"/>
         <geometry>
-          <mesh filename="package://${package_name}/meshes/robot_arms/fr3/visual/link2.dae"/>
+          <mesh filename="package://${package_name}/meshes/visual/link2.dae"/>
         </geometry>
         <material name="">
@@ -153,5 +153,5 @@
         <origin xyz="0 0 0" rpy="0 0 0"/>
         <geometry>
-          <mesh filename="package://${package_name}/meshes/robot_arms/fr3/visual/link3.dae"/>
+          <mesh filename="package://${package_name}/meshes/visual/link3.dae"/>
         </geometry>
         <material name="">
@@ -197,5 +197,5 @@
         <origin xyz="0 0 0" rpy="0 0 0"/>
         <geometry>
-          <mesh filename="package://${package_name}/meshes/robot_arms/fr3/visual/link4.dae"/>
+          <mesh filename="package://${package_name}/meshes/visual/link4.dae"/>
         </geometry>
         <material name="">
@@ -241,5 +241,5 @@
         <origin xyz="0 0 0" rpy="0 0 0"/>
         <geometry>
-          <mesh filename="package://${package_name}/meshes/robot_arms/fr3/visual/link5.dae"/>
+          <mesh filename="package://${package_name}/meshes/visual/link5.dae"/>
         </geometry>
         <material name="">
@@ -303,5 +303,5 @@
         <origin xyz="0 0 0" rpy="0 0 0"/>
         <geometry>
-          <mesh filename="package://${package_name}/meshes/robot_arms/fr3/visual/link6.dae"/>
+          <mesh filename="package://${package_name}/meshes/visual/link6.dae"/>
         </geometry>
         <material name="">
@@ -347,5 +347,5 @@
         <origin xyz="0 0 0" rpy="0 0 0"/>
         <geometry>
-          <mesh filename="package://${package_name}/meshes/robot_arms/fr3/visual/link7.dae"/>
+          <mesh filename="package://${package_name}/meshes/visual/link7.dae"/>
         </geometry>
         <material name="">
